File: new_hardware/freedom_fighter/pif/FreedomFighterPif.sch (EAGLE design)
At the start: 53 parts, among them U1 PIA6821, U10 74LS74D, U11 74LS138D, U12 74LS125D, U2 HM6116P-A, U4 HD68A09EP, U5 74LS74D, U6 74LS245DW, U7 74LS10D, U9 74LS04D

Commit message: Schematic is "final", but I will be removing stuff from it to make the board so I am saving it
Parts:
- removed C100: Unknown value, SparkFun:CAP1206
- removed C9: 0.001uF, SparkFun:CAP1206
- added R100: 680, SparkFun:RESISTOR1206
Connections:
- net E: now also R100.2; no longer C100.2
- net GND: no longer C9.1
- net N$8: now also C14.2; no longer C9.2
- net VCC: now also R100.1; no longer C100.1, C14.2
Other:
- note added: "I guessed at the values for C14 and L1 by using Star Rider as reference. Probably doesn't matter that much."
- note added: "J1 and J2 are molex style, the same as on Star Rider."
- note added: "NOTE: There is an uninstalled IC (U8) and uninstalled set of pin headers (J3) that look to be leftover from Star Rider's design. I did not bother with these since they were never used. They most likely mirror very closely the Star Rider PIF schematic. A capacitor, C9, is installed, which appears to have been intended to go with U8."
- note added: "This appears to be a strong pull-up resistor. Color code suggests that value is 680, while measuring with a multimeter yields a value of 710 (without desoldering it) so this is probably pretty close."
- note removed: "A resistor or cap connecting 'E' to VCC. Still working on discovering this value."
- note removed: "I partly guessed on the values for C9 and C14, and L1 by using Star Rider as reference."
- note removed: "NOTE: There is an uninstalled IC (U8) and uninstalled set of pin headers (J3) that look to be leftover from Star Rider's design. I did not bother with these since they were never used. They most likely mirror very closely the Star Rider PIF schematic."
- moved on the sheet: C14, C15, L1
Changed lines of the file:
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@@
 <?xml version="1.0" encoding="utf-8"?>
 <!DOCTYPE eagle SYSTEM "eagle.dtd">
-<eagle version="6.6.0">
+<eagle version="6.5.0">
 <drawing>
 <settings>
@@
 <setting verticaltext="up"/>
 </settings>
-<grid distance="0.1" unitdist="inch" unit="inch" style="lines" multiple="1" display="no" altdistance="0.05" altunitdist="inch" altunit="inch"/>
+<grid distance="0.1" unitdist="inch" unit="inch" style="lines" multiple="1" display="no" altdistance="0.01" altunitdist="inch" altunit="inch"/>
 <layers>
 <layer number="1" name="Top" color="4" fill="1" visible="no" active="no"/>
@@
 <part name="U10" library="74xx-us" deviceset="74*74" device="D" technology="LS"/>
 <part name="DB1" library="mpo" deviceset="A32077-ND" device="" value="DB25 (FEMALE)"/>
-<part name="C100" library="SparkFun" deviceset="CAP" device="1206" value="Unknown value"/>
 <part name="P+11" library="SparkFun" deviceset="VCC" device=""/>
 <part name="U3" library="memory" deviceset="27256" device=""/>
@@
 <part name="GND5" library="SparkFun" deviceset="GND" device=""/>
 <part name="P+13" library="SparkFun" deviceset="VCC" device=""/>
-<part name="C9" library="SparkFun" deviceset="CAP" device="1206" value="0.001uF"/>
 <part name="C14" library="SparkFun" deviceset="CAP" device="1206" value="0.001uF"/>
 <part name="C15" library="SparkFun" deviceset="CAP_POL" device="PTH2" value="100uF/25V"/>
@@
 <part name="JP8" library="pinhead" deviceset="PINHD-1X7" device=""/>
 <part name="L1" library="SparkFun" deviceset="INDUCTOR" device="H*" technology="1206" value="2.2uH"/>
+<part name="R100" library="SparkFun" deviceset="RESISTOR" device="1206" value="680"/>
 </parts>
 <sheets>
@@
 They most likely mirror
 very closely the Star
-Rider PIF schematic.</text>
+Rider PIF schematic.
+A capacitor, C9, is installed, which appears to
+have been intended to go with U8.</text>
 <text x="233.68" y="-160.02" size="1.778" layer="91">NOTE: DAV' is unconnected.
 This is opposite of Firefox,
@@
 mirror the Star Rider PIF board,
 which is not reflected here.</text>
-<text x="7.62" y="25.4" size="1.778" layer="91">I partly guessed on the values for C9 and C14,
-and L1 by using Star Rider as reference.</text>
+<text x="12.7" y="25.4" size="1.778" layer="91">I guessed at the values for C14
+and L1 by using Star Rider as reference.
+Probably doesn't matter that much.</text>
 <wire x1="31.75" y1="40.64" x2="19.05" y2="40.64" width="0.1524" layer="98" style="longdash"/>
 <wire x1="19.05" y1="40.64" x2="19.05" y2="93.98" width="0.1524" layer="98" style="longdash"/>
@@
 Pins 16-17 are N/C
 from what I can tell.</text>
-<text x="281.94" y="104.14" size="1.778" layer="91">A resistor or cap connecting 'E' to VCC.
-Still working on discovering this value.</text>
+<text x="279.4" y="101.6" size="1.778" layer="91">This appears to be a strong pull-up resistor.
+Color code suggests that value is 680,
+while measuring with a multimeter yields a value of 710 (without desoldering it)
+so this is probably pretty close.</text>
+<text x="-28.956" y="34.544" size="1.778" layer="91">J1 and J2 are
+molex style, the
+same as on Star Rider.</text>
 </plain>
 <instances>
@@
 <instance part="U10" gate="B" x="165.1" y="-40.64"/>
 <instance part="DB1" gate="G$1" x="248.92" y="-129.54"/>
-<instance part="C100" gate="G$1" x="274.32" y="101.6"/>
-<instance part="P+11" gate="1" x="274.32" y="109.22"/>
+<instance part="P+11" gate="1" x="274.32" y="111.76"/>
 <instance part="U3" gate="A" x="198.12" y="68.58"/>
 <instance part="R10" gate="G$1" x="111.76" y="55.88" rot="R270"/>
@@
 <instance part="GND5" gate="1" x="73.66" y="-33.02"/>
 <instance part="P+13" gate="1" x="73.66" y="-15.24"/>
-<instance part="C9" gate="G$1" x="15.24" y="17.78"/>
-<instance part="C14" gate="G$1" x="38.1" y="17.78"/>
-<instance part="C15" gate="G$1" x="63.5" y="17.78" rot="R180"/>
-<instance part="P+14" gate="1" x="73.66" y="15.24" rot="R270"/>
-<instance part="GND1" gate="1" x="76.2" y="22.86" rot="R90"/>
+<instance part="C14" gate="G$1" x="15.24" y="17.78"/>
+<instance part="C15" gate="G$1" x="50.8" y="17.78" rot="R180"/>
+<instance part="P+14" gate="1" x="60.96" y="15.24" rot="R270"/>
+<instance part="GND1" gate="1" x="63.5" y="22.86" rot="R90"/>
 <instance part="R11" gate="G$1" x="144.78" y="-25.4" rot="R270"/>
 <instance part="P+15" gate="1" x="144.78" y="-17.78"/>
@@
 <instance part="P+27" gate="1" x="365.76" y="50.8"/>
 <instance part="C5" gate="G$1" x="365.76" y="43.18" rot="MR0"/>
-<instance part="L1" gate="G$1" x="27.94" y="7.62" rot="R90"/>
+<instance part="L1" gate="G$1" x="30.48" y="7.62" rot="R90"/>
+<instance part="R100" gate="G$1" x="274.32" y="104.14" rot="R270"/>
 </instances>
 <busses>
@@
 </segment>
 <segment>
-<wire x1="10.16" y1="22.86" x2="15.24" y2="22.86" width="0.1524" layer="91"/>
-<pinref part="C9" gate="G$1" pin="1"/>
 <pinref part="J1" gate="-2" pin="S"/>
 <wire x1="7.62" y1="17.78" x2="10.16" y2="17.78" width="0.1524" layer="91"/>
 <wire x1="10.16" y1="17.78" x2="10.16" y2="22.86" width="0.1524" layer="91"/>
 <pinref part="C14" gate="G$1" pin="1"/>
-<wire x1="15.24" y1="22.86" x2="38.1" y2="22.86" width="0.1524" layer="91"/>
+<wire x1="10.16" y1="22.86" x2="15.24" y2="22.86" width="0.1524" layer="91"/>
+<pinref part="GND1" gate="1" pin="GND"/>
+<wire x1="15.24" y1="22.86" x2="50.8" y2="22.86" width="0.1524" layer="91"/>
 <junction x="15.24" y="22.86"/>
-<pinref part="GND1" gate="1" pin="GND"/>
-<wire x1="38.1" y1="22.86" x2="63.5" y2="22.86" width="0.1524" layer="91"/>
-<junction x="38.1" y="22.86"/>
 <pinref part="C15" gate="G$1" pin="-"/>
-<wire x1="63.5" y1="22.86" x2="73.66" y2="22.86" width="0.1524" layer="91"/>
-<junction x="63.5" y="22.86"/>
+<wire x1="50.8" y1="22.86" x2="60.96" y2="22.86" width="0.1524" layer="91"/>
+<junction x="50.8" y="22.86"/>
 </segment>
 <segment>
@@
 <segment>
 <pinref part="P+11" gate="1" pin="VCC"/>
-<pinref part="C100" gate="G$1" pin="1"/>
-<wire x1="274.32" y1="109.22" x2="274.32" y2="106.68" width="0.1524" layer="91"/>
+<pinref part="R100" gate="G$1" pin="1"/>
+<wire x1="274.32" y1="111.76" x2="274.32" y2="109.22" width="0.1524" layer="91"/>
 </segment>
 <segment>
@@
 </segment>
 <segment>
-<pinref part="C14" gate="G$1" pin="2"/>
 <pinref part="P+14" gate="1" pin="VCC"/>
-<wire x1="38.1" y1="15.24" x2="63.5" y2="15.24" width="0.1524" layer="91"/>
 <pinref part="C15" gate="G$1" pin="+"/>
-<wire x1="63.5" y1="15.24" x2="73.66" y2="15.24" width="0.1524" layer="91"/>
-<junction x="63.5" y="15.24"/>
-<wire x1="35.56" y1="7.62" x2="38.1" y2="7.62" width="0.1524" layer="91"/>
-<wire x1="38.1" y1="7.62" x2="38.1" y2="15.24" width="0.1524" layer="91"/>
-<junction x="38.1" y="15.24"/>
+<wire x1="50.8" y1="15.24" x2="60.96" y2="15.24" width="0.1524" layer="91"/>
 <pinref part="L1" gate="G$1" pin="2"/>
+<wire x1="38.1" y1="7.62" x2="50.8" y2="7.62" width="0.1524" layer="91"/>
+<wire x1="50.8" y1="7.62" x2="50.8" y2="15.24" width="0.1524" layer="91"/>
+<junction x="50.8" y="15.24"/>
 </segment>
 <segment>
@@
 <wire x1="259.08" y1="76.2" x2="274.32" y2="76.2" width="0.1524" layer="91"/>
 <label x="261.62" y="76.2" size="1.778" layer="95"/>
-<pinref part="C100" gate="G$1" pin="2"/>
 <wire x1="274.32" y1="76.2" x2="274.32" y2="99.06" width="0.1524" layer="91"/>
 <wire x1="276.86" y1="76.2" x2="274.32" y2="76.2" width="0.1524" layer="91"/>
 <junction x="274.32" y="76.2"/>
+<pinref part="R100" gate="G$1" pin="2"/>
 </segment>
 <segment>
@@
 </segment>
 </net>
-<net name="N$8" class="0">
-<segment>
-<pinref part="C9" gate="G$1" pin="2"/>
-<pinref part="J1" gate="-1" pin="S"/>
-<wire x1="7.62" y1="15.24" x2="15.24" y2="15.24" width="0.1524" layer="91"/>
-<wire x1="20.32" y1="7.62" x2="15.24" y2="7.62" width="0.1524" layer="91"/>
-<wire x1="15.24" y1="7.62" x2="15.24" y2="15.24" width="0.1524" layer="91"/>
-<junction x="15.24" y="15.24"/>
-<pinref part="L1" gate="G$1" pin="1"/>
-</segment>
-</net>
 <net name="N$3" class="0">
 <segment>
 <wire x1="-2.54" y1="5.08" x2="-2.54" y2="33.02" width="0.1524" layer="91"/>
-<wire x1="-2.54" y1="33.02" x2="81.28" y2="33.02" width="0.1524" layer="91"/>
-<wire x1="81.28" y1="33.02" x2="81.28" y2="5.08" width="0.1524" layer="91"/>
-<wire x1="81.28" y1="5.08" x2="-2.54" y2="5.08" width="0.1524" layer="91"/>
+<wire x1="-2.54" y1="33.02" x2="68.58" y2="33.02" width="0.1524" layer="91"/>
+<wire x1="68.58" y1="33.02" x2="68.58" y2="5.08" width="0.1524" layer="91"/>
+<wire x1="68.58" y1="5.08" x2="-2.54" y2="5.08" width="0.1524" layer="91"/>
 </segment>
 </net>
@@
 </segment>
 </net>
+<net name="N$8" class="0">
+<segment>
+<pinref part="C14" gate="G$1" pin="2"/>
+<pinref part="J1" gate="-1" pin="S"/>
+<wire x1="7.62" y1="15.24" x2="15.24" y2="15.24" width="0.1524" layer="91"/>
+<wire x1="22.86" y1="7.62" x2="15.24" y2="7.62" width="0.1524" layer="91"/>
+<wire x1="15.24" y1="7.62" x2="15.24" y2="15.24" width="0.1524" layer="91"/>
+<pinref part="L1" gate="G$1" pin="1"/>
+<junction x="15.24" y="15.24"/>
+</segment>
+</net>

Commit message: completed about half of the routing.  I'd say the hard part is done.
Parts:
- removed C5: 0.1uF, SparkFun:CAP1206
- removed C6: Not Installed, SparkFun:CAP1206
- removed R7, R8: 4.7k, SparkFun:RESISTOR1206
- removed U5: 74LS74D, 74xx-us:74LS74D
Connections:
- removed net !IRQA/FIRQ: JP1.4, R3.2, U1.38, U4.4
- removed net !IRQB/NMI: JP1.2, R5.2, U1.37, U4.2
- removed net 4MS: C6.1, J2-13.S, R8.2, U5B.CLK
- removed net N$1: R7.2, U5A.CLR, U5A.PRE, U5B.CLR
- removed net N$2: U5A.!Q, U5B.D
- new net !FIRQ: JP1.4, R3.2, U4.4
- new net !NMI: JP1.2, R5.2, U4.2
- net !IRQ: no longer U5B.Q
- net D0: no longer U5A.D
- net EVEN/!ODD: no longer J2-15.S, U9B.I
- net GND: no longer C5.2, C6.2, U5B.PRE
- net VCC: no longer C5.1, R7.1, R8.1
Other:
- note removed: "N/C?"
- note removed: "This circuit is installed but does nothing because pin 10 is grounded"
- moved on the sheet: R3

Commit message: 3/4 of the way finished, about to add ground plane
Parts:
- JP5: device pinhead:PINHD-1X8 -> pinhead:PINHD-1X2
Connections:
- net !ENABLE_ROM_E_TO_F: now also JP5.1; no longer JP5.7
- net GND: now also JP5.2; no longer JP5.8
Changed lines of the file:
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@@
 <part name="JP1" library="pinhead" deviceset="PINHD-1X20" device=""/>
 <part name="JP4" library="pinhead" deviceset="PINHD-1X20" device=""/>
-<part name="JP5" library="pinhead" deviceset="PINHD-1X8" device=""/>
 <part name="JP6" library="pinhead" deviceset="PINHD-1X8" device=""/>
 <part name="JP7" library="pinhead" deviceset="PINHD-1X7" device=""/>
@@
 <part name="L1" library="SparkFun" deviceset="INDUCTOR" device="H*" technology="1206" value="2.2uH"/>
 <part name="R100" library="SparkFun" deviceset="RESISTOR" device="1206" value="680"/>
+<part name="JP5" library="pinhead" deviceset="PINHD-1X2" device=""/>
 </parts>
 <sheets>
@@
 <instance part="JP1" gate="A" x="73.66" y="96.52"/>
 <instance part="JP4" gate="A" x="101.6" y="96.52"/>
-<instance part="JP5" gate="A" x="154.94" y="109.22"/>
 <instance part="JP6" gate="A" x="154.94" y="78.74"/>
 <instance part="JP7" gate="A" x="236.22" y="111.76"/>
 <instance part="JP8" gate="A" x="236.22" y="83.82"/>
+<instance part="JP5" gate="G$1" x="154.94" y="101.6"/>
 </instances>
 <busses>
@@
 </segment>
 <segment>
-<pinref part="JP5" gate="A" pin="8"/>
 <wire x1="152.4" y1="101.6" x2="137.16" y2="101.6" width="0.1524" layer="91"/>
 <label x="137.16" y="101.6" size="1.778" layer="95"/>
+<pinref part="JP5" gate="G$1" pin="2"/>
 </segment>
 <segment>
@@
 <net name="!ENABLE_ROM_E_TO_F" class="0">
 <segment>
-<pinref part="JP5" gate="A" pin="7"/>
 <wire x1="152.4" y1="104.14" x2="119.38" y2="104.14" width="0.1524" layer="91"/>
 <label x="119.38" y="104.14" size="1.778" layer="95"/>
-</segment>
-</net>
+<pinref part="JP5" gate="G$1" pin="1"/>
+</segment>
+</net>
