File: new_hardware/freedom_fighter/pif/FreedomFighterPif.sch (EAGLE design)
At the start: 47 parts, among them U1 PIA6821, U10 74LS74D, U11 74LS138D, U12 74LS125D, U2 HM6116P-A, U4 HD68A09EP, U6 74LS245DW, U7 74LS10D, U9 74LS04D

Commit message: updated schematic with notes from measurements
Other:
- note added: "C14 and C15 are confirmed. C14 measured 1078pF (0.001078uF). I guessed at the value for L1 by using Star Rider as reference. Probably doesn't matter that much."
- note added: "This is a strong pull-up resistor. Color code suggests that value is 680, while measuring it (desoldered) yields a value of 710-714."
- note removed: "I guessed at the values for C14 and L1 by using Star Rider as reference. Probably doesn't matter that much."
- note removed: "This appears to be a strong pull-up resistor. Color code suggests that value is 680, while measuring with a multimeter yields a value of 710 (without desoldering it) so this is probably pretty close."
Changed lines of the file:
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@@
 mirror the Star Rider PIF board,
 which is not reflected here.</text>
-<text x="12.7" y="25.4" size="1.778" layer="91">I guessed at the values for C14
-and L1 by using Star Rider as reference.
+<text x="12.7" y="25.4" size="1.778" layer="91">C14 and C15 are confirmed.
+C14 measured 1078pF (0.001078uF).
+I guessed at the value for
+L1 by using Star Rider as reference.
 Probably doesn't matter that much.</text>
 <wire x1="31.75" y1="40.64" x2="19.05" y2="40.64" width="0.1524" layer="98" style="longdash"/>
@@
 Pins 16-17 are N/C
 from what I can tell.</text>
-<text x="279.4" y="101.6" size="1.778" layer="91">This appears to be a strong pull-up resistor.
+<text x="279.4" y="101.6" size="1.778" layer="91">This is a strong pull-up resistor.
 Color code suggests that value is 680,
-while measuring with a multimeter yields a value of 710 (without desoldering it)
-so this is probably pretty close.</text>
+while measuring it (desoldered)
+yields a value of 710-714.</text>
 <text x="-28.956" y="34.544" size="1.778" layer="91">J1 and J2 are
 molex style, the
