File: new_hardware/freedom_fighter/pif/FreedomFighterPif.brd (EAGLE design)
At the start: 160 x 114.3 mm, 47 parts, among them U1 PIA6821, U10 74LS74D, U11 74LS138D, U12 74LS125D, U2 HM6116P-A, U4 HD68A09EP, U6 74LS245DW, U7 74LS10D, U9 74LS04D

Commit message: about to submit v1
Parts:
- moved C13 46.3 mm to (117.2, 14.3), turned to 180 degrees
- moved C12 42.9 mm to (109.5, 15.2), turned to 90 degrees
- moved R5 39.9 mm to (101.6, 74.9), turned to 270 degrees
- moved R6 38.1 mm to (99.1, 72.4), turned to 270 degrees
- moved R9 34.2 mm to (128.3, 81.3)
- moved C4 31.4 mm to (100.3, 66.0), turned to 180 degrees
- moved R100 23.7 mm to (134.6, 62.2), turned to 270 degrees
- moved R3 23.0 mm to (96.5, 71.1)
- moved R4 18.3 mm to (132.1, 80.0), turned to 180 degrees
- moved JP5 9.40 mm to (94.6, 16.8), turned to 90 degrees
- moved U12 7.41 mm to (124.5, 11.4), turned to 0 degrees
- moved JP6 6.35 mm to (105.4, 8.89), turned to 180 degrees
- moved U11 2.54 mm to (101.6, 15.2), turned to 180 degrees
- moved R12 1.27 mm to (92.7, 71.1)
Routing:
- net VCC: track 384.2 -> 558.8 mm, vias 11 -> 15
- net R/!W: track 139.8 -> 230.0 mm, vias 5 -> 9
- net !ENABLE_ROM: track 43.7 -> 104.9 mm, vias 1 -> 4
- net !ENABLE_RAM: track 73.7 -> 130.0 mm, vias 5 -> 9
- net !ENABLE_ROM_E_TO_F: track 0.00 -> 54.3 mm, vias 0 -> 1
- net !RESET: track 133.0 -> 181.6 mm, vias 5 -> 6
- net VP931_DAV: track 61.4 -> 107.1 mm, vias 1 -> 3
- net !ENABLE_VP931_DATA: track 82.5 -> 124.8 mm, vias 7 -> 10
- net !ENABLE_PIA: track 59.1 -> 97.4 mm
- net VP931_DAK: track 63.0 -> 101.0 mm
- net A15: track 5.08 -> 41.5 mm, vias 0 -> 1
- net !ENABLE_ROM_C_TO_D: track 0.00 -> 35.6 mm, vias 0 -> 2
- net A14: track 5.08 -> 38.7 mm, vias 0 -> 1
- net !ENABLE_DAVDAK: track 0.00 -> 32.4 mm, vias 0 -> 2
- net D7: track 150.1 -> 182.4 mm, vias 6 -> 9
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- added copper zone on layer 1, net GND
- added copper zone on layer 16, net GND
Other:
- board size 160 x 114.3 mm -> 138.4 x 114.3 mm
